File: STLINK-adapter.kicad_sch (KiCad schematic)
At the start: 26 parts, among them J1 Conn_02x03_Odd_Even, J2 Conn_01x10, J3 Conn_01x06_Pin

Commit message: added comp values
Parts:
- C1, C2, C3, C4, C5, C6: value C -> 1u
- R1: value R -> 300
- R2: value R -> 200
- R3: value R -> 250
- R4: value R -> 0
